File: Phase_B/PCB_Design/V1/Phase_B_Prototype/Phase_B_Prototype.kicad_sch (KiCad schematic)
At the start: 29 parts, among them J1 USB_B_Mini, U1 CA56-12EWA, U2 74HC595, U3 ATmega32U4-A, Y1 Crystal_GND24

Commit message: Phase B has received a template. Phase A unchanged.
Parts:
- added J2: AVR-ISP-6, symbol Connector:AVR-ISP-6
- added J4: Conn_02x04_Odd_Even, symbol Connector_Generic:Conn_02x04_Odd_Even
- added R15, R16: 330, Resistor_SMD:R_0603_1608Metric, symbol Device:R_Small
- added R17: 10k, Resistor_SMD:R_0603_1608Metric, symbol Device:R_Small
- added U4: USBLC6-2SC6, Package_TO_SOT_SMD:SOT-23-6, symbol Power_Protection:USBLC6-2SC6
Connections:
- net +3.3V: now also J4.4 (Pin_4), J4.6 (Pin_6), J4.8 (Pin_8), R17.1
- net +5V: now also J2.2 (VCC), U4.5 (VBUS)
- net GND: now also J2.6 (GND), J4.1 (Pin_1), U4.2 (GND)
- net Reset: now also J2.5 (~{RST})
- net at J1.2 (D-): now also R16.1
- net at J1.3 (D+): now also R15.1
- net USB_D-: now reaches U3.3 (D-)
- net USB_D+: now reaches U3.4 (D+)
- new net: J4.5 (Pin_5), R17.2
- new net MISO: J2.1 (MISO)
- new net MOSI: J2.4 (MOSI)
- new net RX: J4.7 (Pin_7)
- new net SCK: J2.3 (SCK)
- new net TX: J4.2 (Pin_2)
- new net USB_CONN_D+: R15.2
- new net USB_CONN_D-: R16.2
- no-connect marks 6 -> 7
Other:
- moved on the sheet: D1, D2, LS1, R3, R4, U3
