File: Phase_D/PCB_Design/V1/V1.kicad_sch (KiCad schematic)
At the start: 2 parts

Commit message: Prototype Update
Parts:
- added R1: R, symbol Device:R
- renumbered RV1 to 10K
Connections:
- net GND: now reaches TH1.1
- net GND: now also 10K.1
- net at TH1.2: now also R1.2
- net +5V: now reaches 10K.3
- new net +3.3V: R1.1
Other:
- moved on the sheet: 10K, TH1
Changed lines of the file:
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@@
 (kicad_sch (version 20230121) (generator eeschema)
   (paper "A4")
-  (symbol (lib_id "Device:Thermistor_NTC") (at 88.9 74.93 90) (unit 1)
+  (wire (pts (xy 107.95 92.71) (xy 94.615 92.71))
+    (stroke (width 0) (type default))
+  )
+  (wire (pts (xy 107.95 70.485) (xy 107.95 78.74))
+    (stroke (width 0) (type default))
+  )
+  (wire (pts (xy 159.385 92.075) (xy 159.385 87.63))
+    (stroke (width 0) (type default))
+  )
+  (wire (pts (xy 71.755 92.71) (xy 71.755 96.52))
+    (stroke (width 0) (type default))
+  )
+  (wire (pts (xy 148.59 92.075) (xy 159.385 92.075))
+    (stroke (width 0) (type default))
+  )
+  (wire (pts (xy 86.995 92.71) (xy 71.755 92.71))
+    (stroke (width 0) (type default))
+  )
+  (wire (pts (xy 107.95 86.36) (xy 107.95 92.71))
+    (stroke (width 0) (type default))
+  )
+  (wire (pts (xy 130.175 92.075) (xy 130.175 93.98))
+    (stroke (width 0) (type default))
+  )
+  (wire (pts (xy 140.97 92.075) (xy 130.175 92.075))
+    (stroke (width 0) (type default))
+  )
+  (symbol (lib_id "Device:Thermistor_NTC") (at 90.805 92.71 90) (unit 1)
     (in_bom yes) (on_board yes) (dnp no) (fields_autoplaced)
-    (property "Reference" "TH1" (at 89.2175 69.85 90)
+    (property "Reference" "TH1" (at 91.1225 87.63 90)
       (effects (font (size 1.27 1.27)))
     )
-    (property "Value" "Thermistor_NTC" (at 89.2175 72.39 90)
+    (property "Value" "Thermistor_NTC" (at 91.1225 90.17 90)
       (effects (font (size 1.27 1.27)))
     )
-    (property "Footprint" "" (at 87.63 74.93 0)
+    (property "Footprint" "" (at 89.535 92.71 0)
       (effects (font (size 1.27 1.27)) hide)
     )
-    (property "Datasheet" "~" (at 87.63 74.93 0)
+    (property "Datasheet" "~" (at 89.535 92.71 0)
       (effects (font (size 1.27 1.27)) hide)
     )
@@
     )
   )
-  (symbol (lib_id "Device:R_Potentiometer") (at 144.78 91.44 0) (unit 1)
+  (symbol (lib_id "Device:R_Potentiometer") (at 144.78 92.075 90) (unit 1)
     (in_bom yes) (on_board yes) (dnp no) (fields_autoplaced)
-    (property "Reference" "RV1" (at 142.24 90.805 0)
-      (effects (font (size 1.27 1.27)) (justify right))
+    (property "Reference" "10K" (at 144.78 95.25 90)
+      (effects (font (size 1.27 1.27)))
     )
-    (property "Value" "R_Potentiometer" (at 142.24 93.345 0)
-      (effects (font (size 1.27 1.27)) (justify right))
+    (property "Value" "R_Potentiometer" (at 144.78 97.79 90)
+      (effects (font (size 1.27 1.27)))
     )
-    (property "Footprint" "" (at 144.78 91.44 0)
+    (property "Footprint" "" (at 144.78 92.075 0)
       (effects (font (size 1.27 1.27)) hide)
     )
-    (property "Datasheet" "~" (at 144.78 91.44 0)
+    (property "Datasheet" "~" (at 144.78 92.075 0)
       (effects (font (size 1.27 1.27)) hide)
     )
@@
       (project "V1"
         (path "/bf667db7-508f-459e-90e5-7585272ae06a"
-          (reference "RV1") (unit 1)
+          (reference "10K") (unit 1)
         )
       )
+    )
+  )
+  (symbol (lib_id "power:+5V") (at 159.385 87.63 0) (unit 1)
+    (in_bom yes) (on_board yes) (dnp no) (fields_autoplaced)
+    (property "Reference" "#PWR02" (at 159.385 91.44 0)
+      (effects (font (size 1.27 1.27)) hide)
+    )
+    (property "Value" "+5V" (at 159.385 83.82 0)
+      (effects (font (size 1.27 1.27)))
+    )
+    (property "Footprint" "" (at 159.385 87.63 0)
+      (effects (font (size 1.27 1.27)) hide)
+    )
+    (property "Datasheet" "" (at 159.385 87.63 0)
+      (effects (font (size 1.27 1.27)) hide)
+    )
+    (pin "1")
+    (instances
+      (project "V1"
+        (path "/bf667db7-508f-459e-90e5-7585272ae06a"
+          (reference "#PWR02") (unit 1)
+        )
+      )
+    )
+  )
+  (symbol (lib_id "Device:R") (at 107.95 82.55 0) (unit 1)
+    (in_bom yes) (on_board yes) (dnp no) (fields_autoplaced)
+    (property "Reference" "R1" (at 110.49 81.915 0)
+      (effects (font (size 1.27 1.27)) (justify left))
+    )
+    (property "Value" "R" (at 110.49 84.455 0)
+      (effects (font (size 1.27 1.27)) (justify left))
+    )
+    (property "Footprint" "" (at 106.172 82.55 90)
+      (effects (font (size 1.27 1.27)) hide)
+    )
+    (property "Datasheet" "~" (at 107.95 82.55 0)
+      (effects (font (size 1.27 1.27)) hide)
+    )
+    (pin "1")
+    (pin "2")
+    (instances
+      (project "V1"
+        (path "/bf667db7-508f-459e-90e5-7585272ae06a"
+          (reference "R1") (unit 1)
+        )
+      )
+    )
+  )
+  (symbol (lib_id "power:+3.3V") (at 107.95 70.485 0) (unit 1)
+    (in_bom yes) (on_board yes) (dnp no)
+    (property "Reference" "#PWR01" (at 107.95 74.295 0)
+      (effects (font (size 1.27 1.27)) hide)
+    )
+    (property "Value" "+3.3V" (at 108.585 66.04 0)
+      (effects (font (size 1.27 1.27)))
+    )
+    (property "Footprint" "" (at 107.95 70.485 0)
+      (effects (font (size 1.27 1.27)) hide)
+    )
+    (property "Datasheet" "" (at 107.95 70.485 0)
+      (effects (font (size 1.27 1.27)) hide)
+    )
+    (pin "1")
+    (instances
+      (project "V1"
+        (path "/bf667db7-508f-459e-90e5-7585272ae06a"
+          (reference "#PWR01") (unit 1)
+        )
+      )
+    )
+  )
+  (symbol (lib_id "power:GND") (at 130.175 93.98 0) (unit 1)
+    (in_bom yes) (on_board yes) (dnp no) (fields_autoplaced)
+    (property "Reference" "#PWR04" (at 130.175 100.33 0)
+      (effects (font (size 1.27 1.27)) hide)
+    )
+    (property "Value" "GND" (at 130.175 99.06 0)
+      (effects (font (size 1.27 1.27)))
+    )
+    (property "Footprint" "" (at 130.175 93.98 0)
+      (effects (font (size 1.27 1.27)) hide)
+    )
+    (property "Datasheet" "" (at 130.175 93.98 0)
+      (effects (font (size 1.27 1.27)) hide)
+    )
+    (pin "1")
+    (instances
+      (project "V1"
+        (path "/bf667db7-508f-459e-90e5-7585272ae06a"
+          (reference "#PWR04") (unit 1)
+        )
+      )
+    )
+  )
+  (symbol (lib_id "power:GND") (at 71.755 96.52 0) (unit 1)
+    (in_bom yes) (on_board yes) (dnp no) (fields_autoplaced)
+    (property "Reference" "#PWR03" (at 71.755 102.87 0)
+      (effects (font (size 1.27 1.27)) hide)
+    )
+    (property "Value" "GND" (at 71.755 101.6 0)
+      (effects (font (size 1.27 1.27)))
+    )
+    (property "Footprint" "" (at 71.755 96.52 0)
+      (effects (font (size 1.27 1.27)) hide)
+    )
+    (property "Datasheet" "" (at 71.755 96.52 0)
+      (effects (font (size 1.27 1.27)) hide)
+    )
+    (pin "1")
+    (instances
+      (project "V1"
+        (path "/bf667db7-508f-459e-90e5-7585272ae06a"
+          (reference "#PWR03") (unit 1)
+        )
+      )

Commit message: Supporting Doc Update
Parts:
- added J1: USB3_B_Micro, symbol Connector:USB3_B_Micro
- added U1: STM32C031C4Tx, Package_QFP:LQFP-48_7x7mm_P0.5mm, symbol MCU_ST_STM32C0:STM32C031C4Tx
Connections:
- net +5V: now also J1.1 (VBUS)
- net GND: now also J1.5 (GND)
- net ADC_1: now reaches R1.2, TH1.2
- net ADC_1: now also U1.12 (PA1)
- net ADC_2: now reaches 10K.2
- net ADC_2: now also U1.15 (PA4)
- new net: J1.10 (SSRX+), U1.13 (PA2)
- new net: J1.9 (SSRX-), U1.14 (PA3)
Other:
- title: (none) -> Final Project V1
- moved on the sheet: 10K, R1, TH1

Commit message: Phase D Update
Parts:
- added H1, H2, H3, H4: MountingHole, MountingHole:MountingHole_2.1mm, symbol Mechanical:MountingHole
- added J2, J3: Conn_01x40_Socket, Connector_PinSocket_1.27mm:PinSocket_2x50_P1.27mm_Horizontal, symbol Connector:Conn_01x40_Socket
- 10K1: renamed from 10K; footprint (none) -> Potentiometer_SMD:Potentiometer_ACP_CA6-VSMD_Vertical
- R1: footprint (none) -> Resistor_SMD:R_0201_0603Metric
Connections:
- no-connect marks 0 -> 2
Changed lines of the file:
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@@
   (junction (at 146.05 79.375) (diameter 0) (color 0 0 0 0)
   )
+  (no_connect (at 142.875 43.815))
+  (no_connect (at 140.335 43.815))
   (wire (pts (xy 154.94 66.04) (xy 154.94 68.58))
     (stroke (width 0) (type default))
@@
     )
   )
+  (symbol (lib_id "Mechanical:MountingHole") (at 161.925 112.395 0) (unit 1)
+    (in_bom yes) (on_board yes) (dnp no) (fields_autoplaced)
+    (property "Reference" "H4" (at 164.465 111.76 0)
+      (effects (font (size 1.27 1.27)) (justify left))
+    )
+    (property "Value" "MountingHole" (at 164.465 114.3 0)
+      (effects (font (size 1.27 1.27)) (justify left))
+    )
+    (property "Footprint" "MountingHole:MountingHole_2.1mm" (at 161.925 112.395 0)
+      (effects (font (size 1.27 1.27)) hide)
+    )
+    (property "Datasheet" "~" (at 161.925 112.395 0)
+      (effects (font (size 1.27 1.27)) hide)
+    )
+    (instances
+      (project "V1"
+        (path "/bf667db7-508f-459e-90e5-7585272ae06a"
+          (reference "H4") (unit 1)
+        )
+      )
+    )
+  )
   (symbol (lib_id "Device:R_Potentiometer") (at 191.77 78.74 90) (unit 1)
     (in_bom yes) (on_board yes) (dnp no) (fields_autoplaced)
-    (property "Reference" "10K" (at 191.77 81.915 90)
+    (property "Reference" "10K1" (at 191.77 81.915 90)
       (effects (font (size 1.27 1.27)))
     )
@@
       (effects (font (size 1.27 1.27)))
     )
-    (property "Footprint" "" (at 191.77 78.74 0)
+    (property "Footprint" "Potentiometer_SMD:Potentiometer_ACP_CA6-VSMD_Vertical" (at 191.77 78.74 0)
       (effects (font (size 1.27 1.27)) hide)
     )
@@
       (project "V1"
         (path "/bf667db7-508f-459e-90e5-7585272ae06a"
-          (reference "10K") (unit 1)
+          (reference "10K1") (unit 1)
         )
       )
@@
       (effects (font (size 1.27 1.27)) (justify left))
     )
-    (property "Footprint" "" (at 153.162 72.39 90)
+    (property "Footprint" "Resistor_SMD:R_0201_0603Metric" (at 153.162 72.39 90)
       (effects (font (size 1.27 1.27)) hide)
     )
@@
     )
   )
+  (symbol (lib_id "Mechanical:MountingHole") (at 133.985 131.445 0) (unit 1)
+    (in_bom yes) (on_board yes) (dnp no) (fields_autoplaced)
+    (property "Reference" "H3" (at 136.525 130.81 0)
+      (effects (font (size 1.27 1.27)) (justify left))
+    )
+    (property "Value" "MountingHole" (at 136.525 133.35 0)
+      (effects (font (size 1.27 1.27)) (justify left))
+    )
+    (property "Footprint" "MountingHole:MountingHole_2.1mm" (at 133.985 131.445 0)
+      (effects (font (size 1.27 1.27)) hide)
+    )
+    (property "Datasheet" "~" (at 133.985 131.445 0)
+      (effects (font (size 1.27 1.27)) hide)
+    )
+    (instances
+      (project "V1"
+        (path "/bf667db7-508f-459e-90e5-7585272ae06a"
+          (reference "H3") (unit 1)
+        )
+      )
+    )
+  )
+  (symbol (lib_id "Connector:Conn_01x40_Socket") (at 261.62 86.995 0) (unit 1)
+    (in_bom yes) (on_board yes) (dnp no) (fields_autoplaced)
+    (property "Reference" "J3" (at 263.525 87.63 0)
+      (effects (font (size 1.27 1.27)) (justify left))
+    )
+    (property "Value" "Conn_01x40_Socket" (at 263.525 90.17 0)
+      (effects (font (size 1.27 1.27)) (justify left))
+    )
+    (property "Footprint" "Connector_PinSocket_1.27mm:PinSocket_2x50_P1.27mm_Horizontal" (at 261.62 86.995 0)
+      (effects (font (size 1.27 1.27)) hide)
+    )
+    (property "Datasheet" "~" (at 261.62 86.995 0)
+      (effects (font (size 1.27 1.27)) hide)
+    )
+    (pin "1")
+    (pin "10")
+    (pin "11")
+    (pin "12")
+    (pin "13")
+    (pin "14")
+    (pin "15")
+    (pin "16")
+    (pin "17")
+    (pin "18")
+    (pin "19")
+    (pin "2")
+    (pin "20")
+    (pin "21")
+    (pin "22")
+    (pin "23")
+    (pin "24")
+    (pin "25")
+    (pin "26")
+    (pin "27")
+    (pin "28")
+    (pin "29")
+    (pin "3")
+    (pin "30")
+    (pin "31")
+    (pin "32")
+    (pin "33")
+    (pin "34")
+    (pin "35")
+    (pin "36")
+    (pin "37")
+    (pin "38")
+    (pin "39")
+    (pin "4")
+    (pin "40")
+    (pin "5")
+    (pin "6")
+    (pin "7")
+    (pin "8")
+    (pin "9")
+    (instances
+      (project "V1"
+        (path "/bf667db7-508f-459e-90e5-7585272ae06a"
+          (reference "J3") (unit 1)
+        )
+      )
+    )
+  )
   (symbol (lib_id "power:GND") (at 118.745 31.115 0) (unit 1)
     (in_bom yes) (on_board yes) (dnp no) (fields_autoplaced)
@@
         )
       )
+    )
+  )
+  (symbol (lib_id "Mechanical:MountingHole") (at 133.985 121.285 0) (unit 1)
+    (in_bom yes) (on_board yes) (dnp no) (fields_autoplaced)
+    (property "Reference" "H2" (at 136.525 120.65 0)
+      (effects (font (size 1.27 1.27)) (justify left))
+    )
+    (property "Value" "MountingHole" (at 136.525 123.19 0)
+      (effects (font (size 1.27 1.27)) (justify left))
+    )
+    (property "Footprint" "MountingHole:MountingHole_2.1mm" (at 133.985 121.285 0)
+      (effects (font (size 1.27 1.27)) hide)
+    )
+    (property "Datasheet" "~" (at 133.985 121.285 0)
+      (effects (font (size 1.27 1.27)) hide)
+    )
+    (instances
+      (project "V1"
+        (path "/bf667db7-508f-459e-90e5-7585272ae06a"
+          (reference "H2") (unit 1)
+        )
+      )
+    )
+  )
+  (symbol (lib_id "Connector:Conn_01x40_Socket") (at 227.965 86.995 0) (unit 1)
+    (in_bom yes) (on_board yes) (dnp no) (fields_autoplaced)
+    (property "Reference" "J2" (at 229.87 87.63 0)
+      (effects (font (size 1.27 1.27)) (justify left))
+    )
+    (property "Value" "Conn_01x40_Socket" (at 229.87 90.17 0)
+      (effects (font (size 1.27 1.27)) (justify left))
+    )
+    (property "Footprint" "Connector_PinSocket_1.27mm:PinSocket_2x50_P1.27mm_Horizontal" (at 227.965 86.995 0)
+      (effects (font (size 1.27 1.27)) hide)
+    )
+    (property "Datasheet" "~" (at 227.965 86.995 0)
+      (effects (font (size 1.27 1.27)) hide)
+    )
+    (pin "1")
+    (pin "10")
+    (pin "11")
+    (pin "12")
+    (pin "13")
+    (pin "14")
+    (pin "15")
+    (pin "16")
+    (pin "17")
+    (pin "18")
+    (pin "19")
+    (pin "2")
+    (pin "20")
+    (pin "21")
+    (pin "22")
+    (pin "23")
+    (pin "24")
+    (pin "25")
+    (pin "26")
+    (pin "27")
+    (pin "28")
+    (pin "29")
+    (pin "3")
+    (pin "30")
+    (pin "31")
+    (pin "32")
+    (pin "33")
+    (pin "34")
+    (pin "35")
+    (pin "36")
+    (pin "37")
+    (pin "38")
+    (pin "39")
+    (pin "4")
+    (pin "40")
+    (pin "5")
+    (pin "6")
+    (pin "7")
+    (pin "8")
+    (pin "9")
+    (instances
+      (project "V1"
+        (path "/bf667db7-508f-459e-90e5-7585272ae06a"
+          (reference "J2") (unit 1)
+        )
+      )
+    )
+  )
+  (symbol (lib_id "Mechanical:MountingHole") (at 133.35 111.76 0) (unit 1)
+    (in_bom yes) (on_board yes) (dnp no) (fields_autoplaced)
+    (property "Reference" "H1" (at 135.89 111.125 0)
+      (effects (font (size 1.27 1.27)) (justify left))
+    )
+    (property "Value" "MountingHole" (at 135.89 113.665 0)
+      (effects (font (size 1.27 1.27)) (justify left))
+    )
+    (property "Footprint" "MountingHole:MountingHole_2.1mm" (at 133.35 111.76 0)
+      (effects (font (size 1.27 1.27)) hide)
+    )
+    (property "Datasheet" "~" (at 133.35 111.76 0)
+      (effects (font (size 1.27 1.27)) hide)
+    )
+    (instances
+      (project "V1"
+        (path "/bf667db7-508f-459e-90e5-7585272ae06a"
+          (reference "H1") (unit 1)
+        )
+      )
